Commit message: demo

File: urdf/bluerov.urdf (robot description, URDF)
Before this commit: robot vehicle, 1 links, 0 joints
Links:
- removed link camera_dvl2_link
- added link bluerov/base_link; visual mesh filename=file:///home/da/project/ros/catkin_ws/src/orca_meta/launch/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 scale=1 1 1

Commit message: update

File: urdf/bluerov.urdf (robot description, URDF)
Before this commit: robot vehicle, 1 links, 0 joints
Links:
- link bluerov/base_link: geometry visual mesh filename=package://ORB_DVL2/urdf/bluerov2_noprop.dae scale=1 1 1
